File: Xmas.kicad_sch (KiCad schematic)
At the start: 55 parts, among them IC1 STM32C011F6, IC2 TP4056-42, Q1 AO3401A, Q2 CJ3400, SW1 BZCN_TSA007A1518B03, SW2 BZCN_TSA007A1518B03

Commit message: Update PCB
Parts:
- R14: footprint BornaKiCad:R1206 -> BornaKiCad:R0603; symbol BornaLibrary:R1206 -> BornaLibrary:R0603
Connections:
- net BTN2: now also IC1.11 (PA4); no longer IC1.7 (PA0)
Changed lines of the file:
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@@
 	(wire
 		(pts
-			(xy 36.83 57.15) (xy 50.8 57.15)
-		)
-		(stroke
-			(width 0)
-			(type default)
-		)
-	)
-	(wire
-		(pts
 			(xy 107.95 135.89) (xy 113.03 135.89)
 		)
@@
 	(wire
 		(pts
+			(xy 68.58 64.77) (xy 80.01 64.77)
+		)
+		(stroke
+			(width 0)
+			(type default)
+		)
+	)
+	(wire
+		(pts
 			(xy 185.42 26.67) (xy 185.42 36.83)
 		)
@@
 		)
 	)
-	(label "BTN2"
-		(at 36.83 57.15 0)
-		(fields_autoplaced yes)
-		(effects
-			(font
-				(size 1.27 1.27)
-			)
-			(justify left bottom)
-		)
-	)
 	(label "BUZZER"
 		(at 195.58 142.24 0)
@@
 		)
 	)
+	(label "BTN2"
+		(at 80.01 64.77 0)
+		(fields_autoplaced yes)
+		(effects
+			(font
+				(size 1.27 1.27)
+			)
+			(justify left bottom)
+		)
+	)
 	(label "VDD"
 		(at 111.76 25.4 0)
@@
 	)
 	(symbol
-		(lib_id "BornaLibrary:R1206")
+		(lib_id "BornaLibrary:R0603")
 		(at 248.92 109.22 90)
 		(unit 1)
@@
 			)
 		)
-		(property "Footprint" "BornaKiCad:R1206"
+		(property "Footprint" "BornaKiCad:R0603"
 			(at 252.73 109.22 0)
 			(effects

Commit message: Connected uncotected traces/Marina
Parts:
- C3: value 100n -> 10u; footprint BornaKiCad:C0603 -> Borna KiCAD Library:C1206; symbol BornaLibrary:C0603 -> Borna KiCAD Library:C1206
Changed lines of the file:
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@@
 	)
 	(symbol
-		(lib_id "BornaLibrary:C0603")
+		(lib_id "Borna KiCAD Library:C1206")
 		(at 142.24 139.7 90)
 		(unit 1)
@@
 			)
 		)
-		(property "Value" "100n"
+		(property "Value" "10u"
 			(at 143.51 143.51 0)
 			(effects
@@
 			)
 		)
-		(property "Footprint" "BornaKiCad:C0603"
-			(at 147.32 138.43 0)
+		(property "Footprint" "Borna KiCAD Library:C1206"
+			(at 147.32 139.7 0)
 			(effects
 				(font

Commit message: Fixed paths in project files.
Parts:
- C1, C10, C11, C12, C13, C2, C4, C5, C6, C7, C9: footprint BornaKiCad:C0603 -> Borna KiCAD Library:C0603; symbol BornaLibrary:C0603 -> Borna KiCAD Library:C0603
- C8: footprint BornaKiCad:C1206 -> Borna KiCAD Library:C1206; symbol BornaLibrary:C1206 -> Borna KiCAD Library:C1206
- CONN1: footprint BornaKiCad:JST_S2B-PH-SM4-TB -> Borna KiCAD Library:JST_S2B-PH-SM4-TB; symbol BornaLibrary:S2B-PH-SM4-TB -> Borna KiCAD Library:S2B-PH-SM4-TB
- CONN2: footprint BornaKiCad:TYPE-C_16PIN_2MD(073) -> Borna KiCAD Library:TYPE-C_16PIN_2MD(073); symbol BornaLibrary:TYPE-C_16PIN_2MD(073) -> Borna KiCAD Library:TYPE-C_16PIN_2MD(073)
- D1: footprint BornaKiCad:SOD323 -> Borna KiCAD Library:SOD323; symbol BornaLibrary:BAT20JFILM -> Borna KiCAD Library:BAT20JFILM
- IC1: footprint BornaKiCad:TSSOP20 -> Borna KiCAD Library:TSSOP20; symbol BornaLibrary:STM32C011F6 -> Borna KiCAD Library:STM32C011F6
- IC2: footprint BornaKiCad:EMSOP -> Borna KiCAD Library:EMSOP; symbol BornaLibrary:TP4056-42 -> Borna KiCAD Library:TP4056-42
- LED1, LED10, LED11, LED12, LED2, LED3, LED4, LED5, LED6, LED7, LED8, LED9: footprint BornaKiCad:WS2812B-2020 -> Borna KiCAD Library:WS2812B-2020; symbol BornaLibrary:WS2812B-2020 -> Borna KiCAD Library:WS2812B-2020
- LED13: footprint BornaKiCad:LED_0603 -> Borna KiCAD Library:LED_0603; symbol BornaLibrary:LED_0603 -> Borna KiCAD Library:LED_0603
- Q1: footprint BornaKiCad:SOT-23-3L -> Borna KiCAD Library:SOT-23-3L; symbol BornaLibrary:AO3401A -> Borna KiCAD Library:AO3401A
- Q2: footprint BornaKiCad:SOT-23-3L -> Borna KiCAD Library:SOT-23-3L; symbol BornaLibrary:CJ3400 -> Borna KiCAD Library:CJ3400
- R1, R10, R11, R12, R13, R14, R2, R3, R4, R5, R6, R7, R8, R9: footprint BornaKiCad:R0603 -> Borna KiCAD Library:R0603; symbol BornaLibrary:R0603 -> Borna KiCAD Library:R0603
- SPK1: footprint BornaKiCad:MTL-7525 -> Borna KiCAD Library:MTL-7525; symbol BornaLibrary:MLT-7525 -> Borna KiCAD Library:MLT-7525
- SW1, SW2: footprint BornaKiCad:TSA007A1518B03 -> Borna KiCAD Library:TSA007A1518B03; symbol BornaLibrary:BZCN_TSA007A1518B03 -> Borna KiCAD Library:BZCN_TSA007A1518B03
- TP1, TP2, TP3, TP4, TP5: footprint BornaKiCad:TP-1_5mm -> Borna KiCAD Library:TP-1_5mm; symbol BornaLibrary:TP-1_5mm -> Borna KiCAD Library:TP-1_5mm
Connections:
- net GND: now also SW1.PAD, SW2.PAD

Commit message: Update footprints and PCB have 3D models of components
Parts:
- added U1: TPS7A2633DRVR, BornaKiCadLibrary:WSON-6, symbol BornaLibrary:TPS7A2633DRVR
- C1, C10, C11, C12, C13, C2, C4, C5, C6, C7, C9: footprint Borna KiCAD Library:C0603 -> BornaKiCadLibrary:C0603; symbol Borna KiCAD Library:C0603 -> BornaKiCadLibrary:C0603
- C3, C8: footprint Borna KiCAD Library:C1206 -> BornaKiCadLibrary:C1206; symbol Borna KiCAD Library:C1206 -> BornaKiCadLibrary:C1206
- CONN1: footprint Borna KiCAD Library:JST_S2B-PH-SM4-TB -> BornaKiCadLibrary:JST_S2B-PH-SM4-TB; symbol Borna KiCAD Library:S2B-PH-SM4-TB -> BornaKiCadLibrary:S2B-PH-SM4-TB
- CONN2: footprint Borna KiCAD Library:TYPE-C_16PIN_2MD(073) -> BornaKiCadLibrary:TYPE-C_16PIN_2MD(073); symbol Borna KiCAD Library:TYPE-C_16PIN_2MD(073) -> BornaKiCadLibrary:TYPE-C_16PIN_2MD(073)
- D1: footprint Borna KiCAD Library:SOD323 -> BornaKiCadLibrary:SOD323; symbol Borna KiCAD Library:BAT20JFILM -> BornaKiCadLibrary:BAT20JFILM
- IC1: footprint Borna KiCAD Library:TSSOP20 -> BornaKiCadLibrary:TSSOP20; symbol Borna KiCAD Library:STM32C011F6 -> BornaKiCadLibrary:STM32C011F6
- IC2: footprint Borna KiCAD Library:EMSOP -> BornaKiCadLibrary:EMSOP; symbol Borna KiCAD Library:TP4056-42 -> BornaKiCadLibrary:TP4056-42
- LED1, LED10, LED11, LED12, LED2, LED3, LED4, LED5, LED6, LED7, LED8, LED9: footprint Borna KiCAD Library:WS2812B-2020 -> BornaKiCadLibrary:WS2812B-2020; symbol Borna KiCAD Library:WS2812B-2020 -> BornaKiCadLibrary:WS2812B-2020
- LED13: footprint Borna KiCAD Library:LED_0603 -> BornaKiCadLibrary:LED_0603; symbol Borna KiCAD Library:LED_0603 -> BornaKiCadLibrary:LED_0603
- Q1: footprint Borna KiCAD Library:SOT-23-3L -> BornaKiCadLibrary:SOT-23-3L; symbol Borna KiCAD Library:AO3401A -> BornaKiCadLibrary:AO3401A
- Q2: footprint Borna KiCAD Library:SOT-23-3L -> BornaKiCadLibrary:SOT-23-3L; symbol Borna KiCAD Library:CJ3400 -> BornaKiCadLibrary:CJ3400
- R1, R10, R11, R12, R13, R14, R2, R3, R4, R5, R6, R7, R8, R9: footprint Borna KiCAD Library:R0603 -> BornaKiCadLibrary:R0603; symbol Borna KiCAD Library:R0603 -> BornaKiCadLibrary:R0603
- SPK1: footprint Borna KiCAD Library:MTL-7525 -> BornaKiCadLibrary:MTL-7525; symbol Borna KiCAD Library:MLT-7525 -> BornaKiCadLibrary:MLT-7525
- SW1: footprint Borna KiCAD Library:TSA007A1518B03 -> BornaKiCadLibrary:TSA007A1518B03
- SW2: footprint Borna KiCAD Library:TSA007A1518B03 -> BornaKiCadLibrary:TSA007A1518B03; symbol Borna KiCAD Library:BZCN_TSA007A1518B03 -> BornaKiCadLibrary:BZCN_TSA007A1518B03
- TP1, TP3, TP4, TP5: footprint Borna KiCAD Library:TP-1_5mm -> BornaKiCadLibrary:TP-1_5mm; symbol Borna KiCAD Library:TP-1_5mm -> BornaKiCadLibrary:TP-1_5mm
- TP2: footprint Borna KiCAD Library:TP-1_5mm -> BornaKiCadLibrary:TP-1_5mm
Connections:
- net GND: now also U1.5 (GND), U1.TP
- net VDD: now also U1.4 (EN), U1.6 (VIN); no longer C7.2, C8.2, IC1.4 (VDD)
- new net 3V3: C7.2, C8.2, IC1.4 (VDD), U1.1 (OUT)
Other:
- note added: "VOLTAGE REGULATOR"
- moved on the sheet: CONN1, R1, R2
