File: _autosave-Xmas.kicad_sch (KiCad schematic)
At the start: 55 parts, among them IC1 STM32C011F6, IC2 TP4056-42, Q1 AO3401A, Q2 CJ3400, SW1 BZCN_TSA007A1518B03, SW2 BZCN_TSA007A1518B03

Commit message: Everything on the PCB is connected
Parts:
- R14: footprint BornaKiCad:R1206 -> BornaKiCad:R0603; symbol BornaLibrary:R1206 -> BornaLibrary:R0603
Changed lines of the file:
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@@
 	)
 	(symbol
-		(lib_id "BornaLibrary:R1206")
+		(lib_id "BornaLibrary:R0603")
 		(at 248.92 109.22 90)
 		(unit 1)
@@
 			)
 		)
-		(property "Footprint" "BornaKiCad:R1206"
+		(property "Footprint" "BornaKiCad:R0603"
 			(at 252.73 109.22 0)
 			(effects
