File: Xmas.kicad_pcb (KiCad board)
At the start: 2 copper layers, 50 x 60.6 mm, 56 parts, among them IC1 STM32C011F6, IC2 TP4056-42, Q1 AO3401A, Q2 CJ3400, SW1 BZCN_TSA007A1518B03, SW2 BZCN_TSA007A1518B03, U1 TPS7A2633DRVR

Commit message: Added Gerber file
Routing:
- net WS_SUPPLY: track 220.7 -> 221.8 mm
Other:
- board text added: "2024"
- board text added: "Marina Golic"
